File: zencore.kicad_pcb (KiCad board)
At the start: 2 copper layers, 21 x 51 mm, 17 parts, among them J1 Micro_SD_Card, J2 USB_C_Receptacle_USB2.0_16P, SW1 SW_Push, U1 W25Q128JVS, U2 STM32F411CEUx, Y1 Crystal_GND24_Small

Commit message: Worked on the schematic
Parts:
- added C10: 100n, Capacitor_SMD:C_0402_1005Metric, F.Cu at (175.3, 80.8)
- added C11: 10u, Capacitor_SMD:C_0603_1608Metric, F.Cu at (176.3, 76.8)
- added C12: 100n, Capacitor_SMD:C_0402_1005Metric, F.Cu at (176.2, 78.5)
- added C9: 22u, Capacitor_SMD:C_0603_1608Metric, F.Cu at (171.6, 77.8)
- added D1: LED, LED_SMD:LED_0402_1005Metric, F.Cu at (167.7, 81.0)
- added D2: LED, LED_SMD:LED_0402_1005Metric, F.Cu at (167.7, 80.0)
- added D3: LED, LED_SMD:LED_0402_1005Metric, F.Cu at (167.7, 79.0)
- added D4: LED, LED_SMD:LED_0402_1005Metric, F.Cu at (167.7, 78.0)
- added J3: Conn_01x20_Pin, Connector_PinHeader_2.54mm:PinHeader_1x20_P2.54mm_Vertical, B.Cu at (161.6, 70.4)
- added J4: Conn_01x20_Pin, Connector_PinHeader_2.54mm:PinHeader_1x20_P2.54mm_Vertical, B.Cu at (179.6, 70.5)
- added L1: 2.2u, Inductor_SMD:L_0603_1608Metric, F.Cu at (173.3, 80.0)
- added R10: 100k, Resistor_SMD:R_0402_1005Metric, F.Cu at (176.3, 75.2)
- added R4: 100k, Resistor_SMD:R_0402_1005Metric, F.Cu at (175.3, 78.9)
- added R5: 100R, Resistor_SMD:R_0402_1005Metric, F.Cu at (165.9, 81.0)
- added R6: 100R, Resistor_SMD:R_0402_1005Metric, F.Cu at (165.9, 80.0)
- added R7: 100R, Resistor_SMD:R_0402_1005Metric, F.Cu at (165.9, 79.0)
- added R8: 100R, Resistor_SMD:R_0402_1005Metric, F.Cu at (165.9, 78.0)
- added R9: 5.1k, Resistor_SMD:R_0402_1005Metric, F.Cu at (173.8, 99.5)
- added SW2: SW_Push, easyeda2kicad:SW-SMD_L3.9-W3.0-P4.45, F.Cu at (173.4, 105.2)
- added U3: TPS62162DSG, Package_SON:WSON-8-1EP_2x2mm_P0.5mm_EP0.9x1.6mm_ThermalVias, F.Cu at (173.6, 77.7)
- J1: moved to F.Cu
- R1: value 10k -> 5.1k
- SW1: footprint Button_Switch_SMD:SW_SPST_PTS810 -> easyeda2kicad:SW-SMD_L3.9-W3.0-P4.45
- moved R1 12.4 mm to (176.3, 102.3), turned to 180 degrees
- moved C2 8.41 mm to (167.8, 90.3), turned to 0 degrees
- moved C1 8.03 mm to (175.2, 91.8), turned to -90 degrees
- moved C3 7.92 mm to (172.3, 100.9), turned to -90 degrees
- moved R2 7.88 mm to (164.7, 72.2)
- moved R3 7.65 mm to (176.3, 72.4)
- moved C8 7.44 mm to (171.4, 101.4), turned to 90 degrees
- moved C4 7.30 mm to (166.0, 97.4), turned to 90 degrees
- moved Y1 7.12 mm to (168.8, 101.3)
- moved SW1 6.98 mm to (166.9, 105.2)
- moved C6 6.72 mm to (175.2, 93.7), turned to -90 degrees
- moved C5 6.07 mm to (171.9, 99.5), turned to 180 degrees
- moved U1 2.45 mm to (170.0, 86.8)
- moved C7 2.31 mm to (166.3, 101.4), turned to -90 degrees
- moved J2 1.83 mm to (170.5, 71.4)
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Connections:
- J1 pad 2: SD_DAT3/CD -> SD_DAT3
- U1 pad 1: unconnected-(U1-~{CS}-Pad1) -> SPI1_CSB
- U1 pad 2: unconnected-(U1-DO/IO_{1}-Pad2) -> SPI1_MISO
- U1 pad 3: unconnected-(U1-~{WP}/IO_{2}-Pad3) -> QSPI_WPB
- U1 pad 5: unconnected-(U1-DI/IO_{0}-Pad5) -> SPI1_MOSI
- U1 pad 6: unconnected-(U1-CLK-Pad6) -> SPI1_SCLK
- U1 pad 7: unconnected-(U1-~{HOLD}/~{RESET}/IO_{3}-Pad7) -> QSPI_HOLDB
- U2 pad 1: unconnected-(U2-VBAT-Pad1) -> +3V3
- U2 pad 10: unconnected-(U2-PA0-Pad10) -> Net-(U2-PA0)
- U2 pad 15: unconnected-(U2-PA5-Pad15) -> SPI1_SCLK
- U2 pad 16: unconnected-(U2-PA6-Pad16) -> SD_CMD
- U2 pad 17: unconnected-(U2-PA7-Pad17) -> SPI1_MOSI
- U2 pad 28: unconnected-(U2-PB15-Pad28) -> SD_CLK
- U2 pad 29: unconnected-(U2-PA8-Pad29) -> SD_DAT1
- U2 pad 30: unconnected-(U2-PA9-Pad30) -> SD_DAT2
- U2 pad 31: unconnected-(U2-PA10-Pad31) -> QSPI_HOLDB
- U2 pad 32: unconnected-(U2-PA11-Pad32) -> D-
- U2 pad 33: unconnected-(U2-PA12-Pad33) -> D+
- U2 pad 34: unconnected-(U2-PA13-Pad34) -> SWDIO
- U2 pad 37: unconnected-(U2-PA14-Pad37) -> SWCLK
- U2 pad 38: unconnected-(U2-PA15-Pad38) -> SPI1_CSB
- U2 pad 39: unconnected-(U2-PB3-Pad39) -> QSPI_WPB
- U2 pad 40: unconnected-(U2-PB4-Pad40) -> SPI1_MISO
- U2 pad 41: unconnected-(U2-PB5-Pad41) -> SD_DAT3
- U2 pad 43: unconnected-(U2-PB7-Pad43) -> SD_DAT0
- Y1 pad 1: Net-(U2-PH1) -> Net-(U2-PH0)
- Y1 pad 2: unconnected-(Y1-Pad2) -> GND
- Y1 pad 3: Net-(U2-PH0) -> Net-(U2-PH1)
- Y1 pad 4: unconnected-(Y1-Pad4) -> GND

Commit message: Routing done
Parts:
- removed D3, D4: LED, LED_SMD:LED_0402_1005Metric
- removed R8: 100R, Resistor_SMD:R_0402_1005Metric
- R7: value 100R -> 5.1k
- moved R7 16.1 mm to (164.8, 95.1), turned to 90 degrees
- moved R1 4.39 mm to (172.3, 104.1), turned to -90 degrees
- moved D1 2.63 mm to (165.4, 79.8), turned to -90 degrees
- moved SW2 2.09 mm to (175.0, 103.8), turned to -90 degrees
- moved R6 1.71 mm to (166.3, 81.7), turned to -90 degrees
- moved D2 1.40 mm to (166.3, 79.8), turned to -90 degrees
- moved SW1 1.34 mm to (168.3, 105.1)
- moved R9 0.88 mm to (173.3, 100.3), turned to 90 degrees
- moved R5 0.78 mm to (165.4, 81.7), turned to -90 degrees
- moved U1 0.72 mm to (169.4, 86.4)
- moved C3 0.65 mm to (172.3, 101.5)
- moved C6 0.65 mm to (175.8, 93.8)
- moved C4 0.55 mm to (166.0, 97.9)
- moved C10 0.53 mm to (175.3, 81.3)
- moved C5 0.39 mm to (171.9, 99.9)
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Connections:
- J3 pad 10: unconnected-(J3-Pin_10-Pad10) -> PC13
- J3 pad 11: unconnected-(J3-Pin_11-Pad11) -> PC14
- J3 pad 12: unconnected-(J3-Pin_12-Pad12) -> +3V3
- J3 pad 14: unconnected-(J3-Pin_14-Pad14) -> PC15
- J3 pad 15: unconnected-(J3-Pin_15-Pad15) -> NRST
- J3 pad 16: unconnected-(J3-Pin_16-Pad16) -> PA0
- J3 pad 17: unconnected-(J3-Pin_17-Pad17) -> +3V3
- J3 pad 19: unconnected-(J3-Pin_19-Pad19) -> GND
- J3 pad 20: unconnected-(J3-Pin_20-Pad20) -> GND
- J3 pad 4: unconnected-(J3-Pin_4-Pad4) -> PB6
- J3 pad 5: unconnected-(J3-Pin_5-Pad5) -> BOOT0
- J3 pad 6: unconnected-(J3-Pin_6-Pad6) -> PB8
- J3 pad 7: unconnected-(J3-Pin_7-Pad7) -> +3V3
- J3 pad 9: unconnected-(J3-Pin_9-Pad9) -> PB9
- J4 pad 10: unconnected-(J4-Pin_10-Pad10) -> PB10
- J4 pad 11: unconnected-(J4-Pin_11-Pad11) -> PB2
- J4 pad 12: unconnected-(J4-Pin_12-Pad12) -> PB1
- J4 pad 14: unconnected-(J4-Pin_14-Pad14) -> PB0
- J4 pad 15: unconnected-(J4-Pin_15-Pad15) -> PA4
- J4 pad 16: unconnected-(J4-Pin_16-Pad16) -> PA3
- J4 pad 17: unconnected-(J4-Pin_17-Pad17) -> +3V3
- J4 pad 19: unconnected-(J4-Pin_19-Pad19) -> PA2
- J4 pad 20: unconnected-(J4-Pin_20-Pad20) -> PA1
- J4 pad 6: unconnected-(J4-Pin_6-Pad6) -> PB14
- J4 pad 7: unconnected-(J4-Pin_7-Pad7) -> PB13
- J4 pad 9: unconnected-(J4-Pin_9-Pad9) -> PB12
- R1 pad 2: Net-(U2-NRST) -> NRST
- R5 pad 2: unconnected-(R5-Pad2) -> PB6
- R6 pad 2: unconnected-(R6-Pad2) -> PB8
- R7 pad 1: Net-(D3-A) -> BOOT0
- R7 pad 2: unconnected-(R7-Pad2) -> GND
- R9 pad 1: unconnected-(R9-Pad1) -> +3V3
- R9 pad 2: Net-(U2-PA0) -> PA0
- SW1 pad 2: Net-(U2-NRST) -> NRST
- SW2 pad 1: Net-(U2-PA0) -> PA0
- U2 pad 10: Net-(U2-PA0) -> PA0
- U2 pad 11: unconnected-(U2-PA1-Pad11) -> PA1
- U2 pad 12: unconnected-(U2-PA2-Pad12) -> PA2
- U2 pad 13: unconnected-(U2-PA3-Pad13) -> PA3
- U2 pad 14: unconnected-(U2-PA4-Pad14) -> PA4
- U2 pad 18: unconnected-(U2-PB0-Pad18) -> PB0
- U2 pad 19: unconnected-(U2-PB1-Pad19) -> PB1
- U2 pad 2: unconnected-(U2-PC13-Pad2) -> PC13
- U2 pad 20: unconnected-(U2-PB2-Pad20) -> PB2
- U2 pad 21: unconnected-(U2-PB10-Pad21) -> PB10
- U2 pad 25: unconnected-(U2-PB12-Pad25) -> PB12
- U2 pad 26: unconnected-(U2-PB13-Pad26) -> PB13
- U2 pad 27: unconnected-(U2-PB14-Pad27) -> PB14
- U2 pad 3: unconnected-(U2-PC14-Pad3) -> PC14
- U2 pad 4: unconnected-(U2-PC15-Pad4) -> PC15
- U2 pad 42: unconnected-(U2-PB6-Pad42) -> PB6
- U2 pad 44: unconnected-(U2-BOOT0-Pad44) -> BOOT0
- U2 pad 45: unconnected-(U2-PB8-Pad45) -> PB8
- U2 pad 46: unconnected-(U2-PB9-Pad46) -> PB9
- U2 pad 7: Net-(U2-NRST) -> NRST
Routing:
- net +3V3: track 0.00 -> 119.8 mm, vias 0 -> 8
- net GND: track 0.00 -> 45.5 mm, vias 0 -> 42
- net SD_DAT1: track 0.00 -> 36.5 mm, vias 0 -> 2
- net SD_CLK: track 0.00 -> 36.1 mm, vias 0 -> 2
- net SD_DAT2: track 0.00 -> 33.9 mm, vias 0 -> 2
- net SD_DAT3: track 0.00 -> 33.8 mm, vias 0 -> 2
- net SD_CMD: track 0.00 -> 33.8 mm, vias 0 -> 2
- net SD_DAT0: track 0.00 -> 33.7 mm, vias 0 -> 2
- net SWDIO: track 0.00 -> 25.9 mm
- net +5V: track 0.00 -> 25.5 mm, vias 0 -> 2
- net PA1: track 0.00 -> 24.4 mm
- net SWCLK: track 0.00 -> 22.3 mm
- net PB6: track 0.00 -> 22.1 mm
- net PB8: track 0.00 -> 22.0 mm, vias 0 -> 2
- net PA0: track 0.00 -> 21.7 mm
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- added copper zone on B.Cu, net GND
- added copper zone on F.Cu, net GND
