File: zencore.kicad_sch (KiCad schematic)
At the start: 17 parts, among them J1 Micro_SD_Card, J2 USB_C_Receptacle_USB2.0_16P, SW1 SW_Push, U1 W25Q128JVS, U2 STM32F411CEUx, Y1 Crystal_GND24_Small

Commit message: Worked on the schematic
Parts:
- added C10, C12: 100n, Capacitor_SMD:C_0402_1005Metric, symbol Device:C
- added C11: 10u, Capacitor_SMD:C_0603_1608Metric, symbol Device:C
- added C9: 22u, Capacitor_SMD:C_0603_1608Metric, symbol Device:C
- added D1, D2, D3, D4: LED, LED_SMD:LED_0402_1005Metric, symbol Device:LED
- added J3, J4: Conn_01x20_Pin, Connector_PinHeader_2.54mm:PinHeader_1x20_P2.54mm_Vertical, symbol Connector:Conn_01x20_Pin
- added L1: 2.2u, Inductor_SMD:L_0603_1608Metric, symbol Device:L
- added R10, R4: 100k, Resistor_SMD:R_0402_1005Metric, symbol Device:R
- added R5, R6, R7, R8: 100R, Resistor_SMD:R_0402_1005Metric, symbol Device:R
- added R9: 5.1k, Resistor_SMD:R_0402_1005Metric, symbol Device:R
- added SW2: SW_Push, easyeda2kicad:SW-SMD_L3.9-W3.0-P4.45, symbol Switch:SW_Push
- added U3: TPS62162DSG, Package_SON:WSON-8-1EP_2x2mm_P0.5mm_EP0.9x1.6mm_ThermalVias, symbol Regulator_Switching:TPS62162DSG
- R1: value 10k -> 5.1k
- SW1: footprint Button_Switch_SMD:SW_SPST_PTS810 -> easyeda2kicad:SW-SMD_L3.9-W3.0-P4.45
Connections:
- net SD_DAT3/CD is gone; now on net SD_DAT3: J1.2 (DAT3/CD)
- net +3V3: now also U2.1 (VBAT), C10.1, C9.1, J4.5 (Pin_5), L1.2, R4.1, U3.6 (VOS)
- net +5V: now also C11.1, C12.1, J4.1 (Pin_1), J4.2 (Pin_2), R10.1, U3.2 (VIN)
- net D+: now also U2.33 (PA12)
- net D-: now also U2.32 (PA11)
- net GND: now also Y1.2, Y1.4, C10.2, C11.2, C12.2, C9.2, D1.1 (K), D2.1 (K), D3.1 (K), D4.1 (K), J3.13 (Pin_13), J3.18 (Pin_18), J3.3 (Pin_3), J3.8 (Pin_8), J4.13 (Pin_13), J4.18 (Pin_18), J4.3 (Pin_3), J4.8 (Pin_8), SW2.2, U3.1 (PGND), U3.4 (AGND), U3.5 (FB), U3.9 (PAD)
- net SD_CLK: now also U2.28 (PB15)
- net SD_CMD: now also U2.16 (PA6)
- net SD_DAT0: now also U2.43 (PB7)
- net SD_DAT1: now also U2.29 (PA8)
- net SD_DAT2: now also U2.30 (PA9)
- net at C8.2, U2.6 (PH1): now also Y1.3; no longer Y1.1
- net SPI1_CSB: now reaches U1.1 (~{CS})
- net SPI1_CSB: now also U2.38 (PA15)
- net SPI1_MISO: now reaches U1.2 (DO/IO_{1})
- net SPI1_MISO: now also U2.40 (PB4)
- net QSPI_WPB: now reaches U1.3 (~{WP}/IO_{2})
- net QSPI_WPB: now also U2.39 (PB3)
- net SPI1_MOSI: now reaches U1.5 (DI/IO_{0})
- net SPI1_MOSI: now also U2.17 (PA7)
- net SPI1_SCLK: now reaches U1.6 (CLK)
- net SPI1_SCLK: now also U2.15 (PA5)
- net QSPI_HOLDB: now reaches U1.7 (~{HOLD}/~{RESET}/IO_{3})
- net QSPI_HOLDB: now also U2.31 (PA10)
- net at U2.10 (PA0): now also R9.2, SW2.1
- net SWDIO: now reaches U2.34 (PA13)
- net SWDIO: now also J3.1 (Pin_1)
- net SWCLK: now reaches U2.37 (PA14)
- net SWCLK: now also J3.2 (Pin_2)
- net SD_DAT3: now reaches U2.41 (PB5)
- net at C7.2, U2.5 (PH0): now also Y1.1; no longer Y1.3
- new net: L1.1, U3.7 (SW)
- new net: D3.2 (A), R7.1
- new net: D2.2 (A), R6.1
- new net: D1.2 (A), R5.1
- new net: D4.2 (A), R8.1
- new net: R4.2, U3.8 (PG)
- new net 3v3_EN: J4.4 (Pin_4), R10.2, U3.3 (EN)
Other:
- note added: "Buck Converter 5V to 3.3V"
- note added: "USB"
- moved on the sheet: C1, C2, C3, C4, C5, C6, C7, C8, J1, R1, R2, SW1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

Commit message: Routing done
Parts:
- removed D3, D4: LED, LED_SMD:LED_0402_1005Metric, symbol Device:LED
- removed R8: 100R, Resistor_SMD:R_0402_1005Metric, symbol Device:R
- R7: value 100R -> 5.1k
Connections:
- net +3V3: now also J3.12 (Pin_12), J3.17 (Pin_17), J3.8 (Pin_8), J4.17 (Pin_17), R9.1
- net GND: now also J3.19 (Pin_19), J3.20 (Pin_20), J3.7 (Pin_7), R7.2; no longer J3.8 (Pin_8)
- net PA0: now reaches R9.2, SW2.1, U2.10 (PA0)
- net PA0: now also J3.16 (Pin_16)
- net NRST: now reaches R1.2, SW1.2, U2.7 (NRST)
- net NRST: now also J3.15 (Pin_15)
- net BOOT0: now reaches R7.1
- net BOOT0: now also J3.5 (Pin_5), U2.44 (BOOT0)
- net PC13: now reaches J3.10 (Pin_10)
- net PC13: now also U2.2 (PC13)
- net PC14: now reaches J3.11 (Pin_11)
- net PC14: now also U2.3 (PC14)
- net PC15: now reaches J3.14 (Pin_14)
- net PC15: now also U2.4 (PC15)
- net PB6: now reaches J3.4 (Pin_4)
- net PB6: now also R5.2, U2.42 (PB6)
- net PB8: now reaches J3.6 (Pin_6)
- net PB8: now also R6.2, U2.45 (PB8)
- net PB9: now reaches J3.9 (Pin_9)
- net PB9: now also U2.46 (PB9)
- net PB10: now reaches J4.10 (Pin_10)
- net PB10: now also U2.21 (PB10)
- net PB2: now reaches J4.11 (Pin_11)
- net PB2: now also U2.20 (PB2)
- net PB1: now reaches J4.12 (Pin_12)
- net PB1: now also U2.19 (PB1)
- net PB0: now reaches J4.14 (Pin_14)
- net PB0: now also U2.18 (PB0)
- net PA4: now reaches J4.15 (Pin_15)
- net PA4: now also U2.14 (PA4)
- net PA3: now reaches J4.16 (Pin_16)
- net PA3: now also U2.13 (PA3)
- net PA2: now reaches J4.19 (Pin_19)
- net PA2: now also U2.12 (PA2)
- net PA1: now reaches J4.20 (Pin_20)
- net PA1: now also U2.11 (PA1)
- net PB14: now reaches J4.6 (Pin_6)
- net PB14: now also U2.27 (PB14)
- net PB13: now reaches J4.7 (Pin_7)
- net PB13: now also U2.26 (PB13)
- net PB12: now reaches J4.9 (Pin_9)
- net PB12: now also U2.25 (PB12)
